File: GazSensor-Rodier&Xu/GazSensor-Rodier&Xu.kicad_pcb (KiCad board)
At the start: 2 copper layers, 68.6 x 53.3 mm, 15 parts, among them J1 Conn_01x08_Female, J2 Conn_01x02_Female

Commit message: Add files via upload
Parts:
- removed Rsensor1: 10k<...<1G, Package_TO_SOT_THT:TO-5-4
- moved J2 14.0 mm to (132.1, 83.8)
Routing:
- net arduino3v: track 103.2 -> 100.4 mm
- net Net-(J2-Pad2): track 10.8 -> 11.3 mm
Changed lines of the file:
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@@
     (thickness 1.6)
     (drawings 12)
-    (tracks 105)
+    (tracks 104)
     (zones 0)
-    (modules 15)
+    (modules 14)
     (nets 13)
   )
@@
     )
   )
-  (module Package_TO_SOT_THT:TO-5-4 (layer F.Cu)
-    (at 121.92 97.79 90)
-    (descr TO-5-4)
-    (tags TO-5-4)
-    (fp_text reference Rsensor1 (at 8.89 -1.27 180) (layer F.SilkS)
-      (effects (font (size 1 1) (thickness 0.15)))
-    )
-    (fp_text value 10k<...<1G (at -5.08 -2.54 180) (layer F.Fab)
-      (effects (font (size 1 1) (thickness 0.15)))
-    )
-    (fp_text user %R (at -3.81 -1.27 180) (layer F.Fab)
-      (effects (font (size 1 1) (thickness 0.15)))
-    )
-    (fp_line (start -0.465408 -3.61352) (end -1.27151 -4.419621) (layer F.Fab) (width 0.1))
-    (fp_line (start -1.27151 -4.419621) (end -1.879621 -3.81151) (layer F.Fab) (width 0.1))
-    (fp_line (start -1.879621 -3.81151) (end -1.07352 -3.005408) (layer F.Fab) (width 0.1))
-    (fp_line (start -0.457084 -3.774902) (end -1.348039 -4.665856) (layer F.SilkS) (width 0.12))
-    (fp_line (start -1.348039 -4.665856) (end -2.125856 -3.888039) (layer F.SilkS) (width 0.12))
-    (fp_line (start -2.125856 -3.888039) (end -1.234902 -2.997084) (layer F.SilkS) (width 0.12))
-    (fp_line (start -2.41 -4.95) (end -2.41 4.95) (layer F.CrtYd) (width 0.05))
-    (fp_line (start -2.41 4.95) (end 7.49 4.95) (layer F.CrtYd) (width 0.05))
-    (fp_line (start 7.49 4.95) (end 7.49 -4.95) (layer F.CrtYd) (width 0.05))
-    (fp_line (start 7.49 -4.95) (end -2.41 -4.95) (layer F.CrtYd) (width 0.05))
-    (fp_circle (center 2.54 0) (end 6.79 0) (layer F.Fab) (width 0.1))
-    (fp_arc (start 2.54 0) (end -0.465408 -3.61352) (angle 349.5) (layer F.Fab) (width 0.1))
-    (fp_arc (start 2.54 0) (end -0.457084 -3.774902) (angle 346.9) (layer F.SilkS) (width 0.12))
-    (pad 1 thru_hole oval (at 0 0 90) (size 1.6 1.2) (drill 0.7) (layers *.Cu *.Mask))
-    (pad 2 thru_hole oval (at 2.54 2.54 90) (size 1.2 1.2) (drill 0.7) (layers *.Cu *.Mask)
-      (net 1 arduino3v))
-    (pad 3 thru_hole oval (at 5.08 0 90) (size 1.2 1.2) (drill 0.7) (layers *.Cu *.Mask))
-    (pad 4 thru_hole oval (at 2.54 -2.54 90) (size 1.2 1.2) (drill 0.7) (layers *.Cu *.Mask))
-    (model ${KISYS3DMOD}/Package_TO_SOT_THT.3dshapes/TO-5-4.wrl
-      (at (xyz 0 0 0))
-      (scale (xyz 1 1 1))
-      (rotate (xyz 0 0 0))
-    )
-  )
   (module Connector:NS-Tech_Grove_1x04_P2mm_Vertical (layer F.Cu)
     (at 129.54 110.49)
@@
   )
   (module Connector_PinHeader_2.00mm:PinHeader_1x02_P2.00mm_Vertical (layer F.Cu)
-    (at 146.05 83.82)
+    (at 132.08 83.82)
     (descr "Through hole straight pin header, 1x02, 2.00mm pitch, single row")
     (tags "Through hole pin header THT 1x02 2.00mm single row")
@@
     (effects (font (size 0.75 0.75) (thickness 0.1875)))
   )
-  (gr_text 3V (at 128.27 96.52 90) (layer F.Cu)
+  (gr_text 3V (at 132.08 81.28 90) (layer F.Cu)
     (effects (font (size 0.75 0.75) (thickness 0.1875)))
   )
-  (gr_text "Capteur de gaz à connectique \nTO5" (at 114.3 96.52 90) (layer F.Cu)
+  (gr_text "Capteur de gaz à connectique \nTO5" (at 124.46 85.09 90) (layer F.Cu)
     (effects (font (size 0.75 0.75) (thickness 0.1875)))
   )
@@
   (segment (start 155.695001 126.244999) (end 155.695001 120.054999) (width 0.8) (layer F.Cu) (net 1))
   (segment (start 154.609999 127.330001) (end 155.695001 126.244999) (width 0.8) (layer F.Cu) (net 1))
-  (segment (start 135.89 83.82) (end 124.46 95.25) (width 0.8) (layer F.Cu) (net 1))
-  (segment (start 146.05 83.82) (end 135.89 83.82) (width 0.8) (layer F.Cu) (net 1))
-  (segment (start 124.46 96.098528) (end 124.46 95.25) (width 0.8) (layer F.Cu) (net 1))
-  (segment (start 124.46 108.48763) (end 124.46 96.098528) (width 0.8) (layer F.Cu) (net 1))
-  (segment (start 128.46237 112.49) (end 124.46 108.48763) (width 0.8) (layer F.Cu) (net 1))
-  (segment (start 129.54 112.49) (end 128.46237 112.49) (width 0.8) (layer F.Cu) (net 1))
-  (segment (start 146.05 78.74) (end 147.32 77.47) (width 0.8) (layer F.Cu) (net 1))
-  (segment (start 146.05 83.82) (end 146.05 78.74) (width 0.8) (layer F.Cu) (net 1))
+  (segment (start 140.97 83.82) (end 147.32 77.47) (width 0.8) (layer F.Cu) (net 1))
+  (segment (start 132.08 83.82) (end 140.97 83.82) (width 0.8) (layer F.Cu) (net 1))
+  (segment (start 128.46237 112.49) (end 129.54 112.49) (width 0.8) (layer F.Cu) (net 1))
+  (segment (start 127.977999 112.005629) (end 128.46237 112.49) (width 0.8) (layer F.Cu) (net 1))
+  (segment (start 127.977999 86.447001) (end 127.977999 112.005629) (width 0.8) (layer F.Cu) (net 1))
+  (segment (start 130.605 83.82) (end 127.977999 86.447001) (width 0.8) (layer F.Cu) (net 1))
+  (segment (start 132.08 83.82) (end 130.605 83.82) (width 0.8) (layer F.Cu) (net 1))
   (segment (start 154.94 96.52) (end 155.34 96.52) (width 0.8) (layer F.Cu) (net 2))
   (segment (start 168.95 96.52) (end 154.94 96.52) (width 0.8) (layer F.Cu) (net 2))
@@
   (segment (start 164.37 119.38) (end 164.37 118.425406) (width 0.8) (layer F.Cu) (net 10))
   (segment (start 172.72 125.73) (end 166.37 119.38) (width 0.8) (layer F.Cu) (net 11))
-  (segment (start 139.7 92.17) (end 146.05 85.82) (width 0.8) (layer F.Cu) (net 12))
-  (segment (start 139.7 93.98) (end 139.7 92.17) (width 0.8) (layer F.Cu) (net 12))
+  (segment (start 139.7 93.44) (end 139.7 93.98) (width 0.8) (layer F.Cu) (net 12))
+  (segment (start 132.08 85.82) (end 139.7 93.44) (width 0.8) (layer F.Cu) (net 12))
   (zone (net 0) (net_name "") (layer F.Cu) (hatch edge 0.508)
     (connect_pads (clearance 0.508))
@@
     (polygon
       (pts
-        (xy 111.76 128.27) (xy 176.53 128.27) (xy 177.8 127) (xy 177.8 115.57) (xy 180.34 113.03)
-        (xy 180.34 80.01) (xy 177.8 77.47) (xy 177.8 74.93) (xy 111.76 74.93)
+        (xy 111.76 74.93) (xy 177.8 74.93) (xy 177.8 77.47) (xy 180.34 80.01) (xy 180.34 113.03)
+        (xy 177.8 115.57) (xy 177.8 127) (xy 176.53 128.27) (xy 111.76 128.27)
       )
     )
